File: I2C-7-Segment-Backpack-dot36inch.brd (EAGLE design)
At the start: 27.9 x 27.9 mm, 19 parts, among them J1 H4P-SMD-2.0, U1 AS1115

Commit message: Rev C
Other:
- board text added: "I2C-7 SEG (.36") (C)"
- board text added: "I2C-7 Seg (.36") (C)"
- board text added: "dcity.org"
- board text removed: "I2C-7 SEG (.36") (B)"
- board text removed: "I2C-7 Seg (.36") (B)"
- board text removed: "wht.io"
Changed lines of the file:
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@@
 <?xml version="1.0" encoding="utf-8"?>
 <!DOCTYPE eagle SYSTEM "eagle.dtd">
-<eagle version="7.5.0">
+<eagle version="9.1.3">
 <drawing>
 <settings>
 <setting alwaysvectorfont="no"/>
+<setting keepoldvectorfont="yes"/>
 <setting verticaltext="up"/>
 </settings>
@@
 <hole x="3.175" y="3.175" drill="3.175"/>
 <circle x="8.636" y="18.161" radius="0.254" width="0.2032" layer="21"/>
-<text x="6.858" y="0.635" size="0.889" layer="21" font="vector" ratio="15">I2C-7 Seg (.36") (B)</text>
+<text x="6.858" y="0.635" size="0.889" layer="21" font="vector" ratio="15">I2C-7 Seg (.36") (C)</text>
 <text x="10.16" y="26.67" size="0.889" layer="21" font="vector" ratio="15">I2C ADDR JUMPERS</text>
 <text x="10.16" y="22.86" size="0.889" layer="21" font="vector" ratio="15">BOTH OPEN=03h</text>
@@
 <text x="10.16" y="25.4" size="0.889" layer="21" font="vector" ratio="15">3 CLOSED=01h</text>
 <text x="10.16" y="21.59" size="0.889" layer="21" font="vector" ratio="15">DO NOT CLOSE BOTH</text>
-<text x="21.59" y="0.635" size="0.889" layer="22" font="vector" ratio="15" rot="MR0">I2C-7 SEG (.36") (B)</text>
+<text x="21.59" y="0.635" size="0.889" layer="22" font="vector" ratio="15" rot="MR0">I2C-7 SEG (.36") (C)</text>
 <text x="20.32" y="7.747" size="0.889" layer="21" font="vector" ratio="15" rot="R180">LED1</text>
 <text x="12.827" y="7.366" size="0.889" layer="22" font="vector" ratio="15" rot="MR180">LED1</text>
@@
 <rectangle x1="18.669" y1="11.557" x2="19.685" y2="12.954" layer="43"/>
 <rectangle x1="18.669" y1="14.986" x2="19.685" y2="16.51" layer="43"/>
-<text x="1.27" y="6.096" size="1.27" layer="21" font="vector" ratio="10">wht.io</text>
-<text x="12.446" y="2.286" size="1.27" layer="22" font="vector" ratio="10" rot="MR0">wht.io</text>
+<text x="0.381" y="6.35" size="1.27" layer="21" font="vector" ratio="10">dcity.org</text>
+<text x="14.986" y="2.286" size="1.27" layer="22" font="vector" ratio="10" rot="MR0">dcity.org</text>
 <text x="20.955" y="21.717" size="0.889" layer="22" font="vector" ratio="14" rot="MR0">1 = SDA PULLUP
 2 = SCL PULLUP
@@
 <param name="dpMaxLengthDifference" value="10mm"/>
 <param name="dpGapFactor" value="2.5"/>
-<param name="checkGrid" value="0"/>
 <param name="checkAngle" value="1"/>
 <param name="checkFont" value="1"/>
 <param name="checkRestrict" value="1"/>
+<param name="checkStop" value="0"/>
+<param name="checkValues" value="0"/>
+<param name="checkNames" value="1"/>
+<param name="checkWireStubs" value="1"/>
+<param name="checkPolygonWidth" value="0"/>
 <param name="useDiameter" value="13"/>
 <param name="maxErrors" value="50"/>
@@
 </signal>
 </signals>
+<mfgpreviewcolors>
+<mfgpreviewcolor name="soldermaskcolor" color="0xC8008000"/>
+<mfgpreviewcolor name="silkscreencolor" color="0xFFFEFEFE"/>
+<mfgpreviewcolor name="backgroundcolor" color="0xFF282828"/>
+<mfgpreviewcolor name="coppercolor" color="0xFFFFBF00"/>
+<mfgpreviewcolor name="substratecolor" color="0xFF786E46"/>
+</mfgpreviewcolors>
 </board>
 </drawing>

Commit message: Rev D
Parts:
- added J2: QWIIC_RIGHT_ANGLE, 0:JST04_1MM_RA
- J1: value H4P-SMD-2.0 -> QWIIC_RIGHT_ANGLE; device 0:HW4-SMD-2.0 -> 0:JST04_1MM_RA
- moved J1 4.02 mm to (22.9, 10.2), turned to 90 degrees
Connections:
- net GND: now also J1.1, J2.1; no longer J1.4
- net SCL: now also J1.4, J2.4; no longer J1.1
- net SDA: now also J1.3, J2.3; no longer J1.2
- net VCC: now also J1.2, J2.2; no longer J1.3
Routing:
- net VCC: track 53.1 -> 66.5 mm
- net N$8: track 27.4 -> 16.8 mm, vias 2 -> 1
- net SDA: track 33.2 -> 40.8 mm, vias 0 -> 3
- net SCL: track 42.8 -> 49.3 mm, vias 3 -> 5
- net GND: track 18.5 -> 23.2 mm, vias 4 -> 3
- net N$5: track 20.3 -> 19.3 mm
Other:
- board text added: "I2C-7 SEG (.36") (D)"
- board text added: "I2C-7 Seg (.36") (D)"
- board text removed: "I2C-7 SEG (.36") (C)"
- board text removed: "I2C-7 Seg (.36") (C)"
