File: I2C-7-Segment-Backpack-dot36inch.sch (EAGLE design)
At the start: 19 parts, among them J1 H4P-SMD-2.0, U1 AS1115

Commit message: Rev D
Parts:
- added J2: QWIIC_RIGHT_ANGLE, 0:QWIIC_CONNECTORJS-1MM
- J1: value H4P-SMD-2.0 -> QWIIC_RIGHT_ANGLE; device 0:GROVE-CONNECTOR-SMD(4+2P-2.0) -> 0:QWIIC_CONNECTORJS-1MM
Connections:
- net GND: now also J1.1, J2.1; no longer J1.4
- net SCL: now also J1.4, J2.4; no longer J1.1
- net SDA: now also J1.3, J2.3; no longer J1.2
- net VCC: now also J1.2, J2.2; no longer J1.3
